File: ecu/ecu.kicad_pcb (KiCad board)
At the start: 2 copper layers, 180 x 50 mm, 162 parts, among them J1 INPUTS, J2 OUTPUTS, J3 DEBUG, J5 OLED, Q1 AOD4185, Q2 AOD4185, Q3 AOD4185, Q4 BXT3800P06M, Q5 BXT3800P06M, Q6 BXT3800P06M, Q7 BXT3800P06M, Q8 AOD4185, SW1 DISP_BUTTON, U1 MCP2551-I-SN, U10 AOZ1282CI-1, U3 SB6286, U4 ULN2003, U5 ULN2003, U6 STM32F103VETx, U7 AMS1117-5.0, U8 78L15MG-AA3-R, U9 FM24CL16B, Y1 16MHz

Commit message: pcb layout completed
Parts:
- C29, C31, SW1: moved to B.Cu
- moved SW1 177.4 mm to (210.5, 135.2), turned to 0 degrees
- moved F2 12.0 mm to (187.2, 136.8)
- moved C31 5.55 mm to (139.2, 120.8)
- moved C29 4.65 mm to (137.5, 125.8)
- moved R38 3.82 mm to (121.2, 105.8), turned to 90 degrees
- moved C47 3.04 mm to (128.0, 145.8)
- moved D23 2.76 mm to (127.8, 141.5)
- moved C33 2.02 mm to (137.8, 112.8), turned to 90 degrees
- moved R55 2.02 mm to (130.0, 140.5)
- moved D24 1.75 mm to (218.2, 144.5)
- moved C1 1.50 mm to (212.2, 144.0)
- moved R58 1.50 mm to (206.5, 142.2)
- moved C36 1.25 mm to (152.0, 131.5)
- moved C35 1.03 mm to (139.0, 132.5)
- moved D1 1.00 mm to (207.0, 129.5)
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Connections:
- C46 pad 1: +3.3V -> +3V3
- J3 pad 1: +3.3V -> +3V3
- J3 pad 2: +3.3V -> +3V3
- R56 pad 1: +3.3V -> +3V3
- R57 pad 1: +3.3V -> +3V3
- U6 pad 1: unconnected-(U6-PE2-Pad1) -> /LED_INDICATOR
- U6 pad 15: unconnected-(U6-PC0-Pad15) -> /LIGHT_HAZARD
- U6 pad 16: unconnected-(U6-PC1-Pad16) -> /LIGHT_DAYTIME
- U6 pad 17: unconnected-(U6-PC2-Pad17) -> /APC
- U6 pad 18: unconnected-(U6-PC3-Pad18) -> /INVERTER
- U6 pad 2: unconnected-(U6-PE3-Pad2) -> /LED_AIRBAG
- U6 pad 20: unconnected-(U6-VREF--Pad20) -> GND
- U6 pad 21: unconnected-(U6-VREF+-Pad21) -> +3V3
- U6 pad 3: unconnected-(U6-PE4-Pad3) -> /LED_ABS
- U6 pad 33: unconnected-(U6-PC4-Pad33) -> /WINDSHIELD_HEAT
- U6 pad 34: unconnected-(U6-PC5-Pad34) -> /WIPERS
- U6 pad 35: unconnected-(U6-PB0-Pad35) -> /BMS
- U6 pad 36: unconnected-(U6-PB1-Pad36) -> /INDIC_LEFT
- U6 pad 37: unconnected-(U6-PB2-Pad37) -> /INDIC_RIGHT
- U6 pad 38: unconnected-(U6-PE7-Pad38) -> /LIGHT_STOP
- U6 pad 39: unconnected-(U6-PE8-Pad39) -> /LIGHT_REVERSE
- U6 pad 4: unconnected-(U6-PE5-Pad4) -> /LED_BELT
- U6 pad 40: unconnected-(U6-PE9-Pad40) -> /HEATING
- U6 pad 41: unconnected-(U6-PE10-Pad41) -> /LED_CHARGING
- U6 pad 42: unconnected-(U6-PE11-Pad42) -> /LED_BATTERY_HV
- U6 pad 43: unconnected-(U6-PE12-Pad43) -> /OLED_POWER_EN
- U6 pad 44: unconnected-(U6-PE13-Pad44) -> /IN_DISP
- U6 pad 45: unconnected-(U6-PE14-Pad45) -> /IN_CEINT
- U6 pad 46: unconnected-(U6-PE15-Pad46) -> /IN_CTL_APC
- U6 pad 47: unconnected-(U6-PB10-Pad47) -> /IN_ECO
- U6 pad 48: unconnected-(U6-PB11-Pad48) -> /IN_WINDSHIELD_HEAT
- U6 pad 5: unconnected-(U6-PE6-Pad5) -> /LED_BRAKE
- U6 pad 51: unconnected-(U6-PB12-Pad51) -> /IN_DRIVE_DIR_1
- U6 pad 52: unconnected-(U6-PB13-Pad52) -> /IN_WIPER
- U6 pad 53: unconnected-(U6-PB14-Pad53) -> /IN_FOG_LIGHT
- U6 pad 54: unconnected-(U6-PB15-Pad54) -> /IN_SIDELIGHTS
- U6 pad 55: unconnected-(U6-PD8-Pad55) -> /IN_BRAKE_1
- U6 pad 56: unconnected-(U6-PD9-Pad56) -> /IN_INDICATOR_RIGHT
- U6 pad 57: unconnected-(U6-PD10-Pad57) -> /LED_SIDELIGHTS
- U6 pad 58: unconnected-(U6-PD11-Pad58) -> /LED_HEADLIGHT
- U6 pad 7: unconnected-(U6-PC13-Pad7) -> /LED_STOP
- U6 pad 8: unconnected-(U6-PC14-Pad8) -> /LED_ELECTR
- U6 pad 83: unconnected-(U6-PD2-Pad83) -> /IN_WINDSHIELD_JET
- U6 pad 84: unconnected-(U6-PD3-Pad84) -> /IN_DRIVE_DIR_2
- U6 pad 85: unconnected-(U6-PD4-Pad85) -> /IN_DF_CONV
- U6 pad 86: unconnected-(U6-PD5-Pad86) -> /IN_PARK
- U6 pad 87: unconnected-(U6-PD6-Pad87) -> /IN_AIRBAG
- U6 pad 88: unconnected-(U6-PD7-Pad88) -> /IN_KEY2
- U6 pad 89: unconnected-(U6-PB3-Pad89) -> /IN_CRASH
- U6 pad 9: unconnected-(U6-PC15-Pad9) -> /LED_TEMP
- U6 pad 90: unconnected-(U6-PB4-Pad90) -> /IN_KEY1
- U6 pad 91: unconnected-(U6-PB5-Pad91) -> /IN_HIGHBEAM
- U6 pad 96: unconnected-(U6-PB9-Pad96) -> /LED_HEATER
- U6 pad 97: unconnected-(U6-PE0-Pad97) -> /LED_FOG
- U6 pad 98: unconnected-(U6-PE1-Pad98) -> /LED_BATTERY
- U9 pad 8: +3.3V -> +3V3
Routing:
- net +5V: track 11.7 -> 151.0 mm, vias 0 -> 3
- net /LED_SIDELIGHTS: track 0.00 -> 91.0 mm
- net /IN_DISP: track 0.00 -> 80.6 mm, vias 0 -> 2
- net /LED_HEADLIGHT: track 0.00 -> 77.7 mm
- net /LED_HEATER: track 0.00 -> 77.6 mm, vias 0 -> 2
- net /IN_AIRBAG: track 11.1 -> 86.3 mm, vias 0 -> 2
- net /IN_CEINT: track 10.8 -> 82.5 mm, vias 0 -> 2
- net /IN_CTL_APC: track 6.02 -> 77.5 mm, vias 0 -> 2
- net /IN_PARK: track 7.08 -> 77.1 mm, vias 0 -> 2
- net /IN_DF_CONV: track 1.52 -> 69.8 mm, vias 0 -> 2
- net /LED_ABS: track 0.00 -> 67.9 mm
- net /IN_ECO: track 3.94 -> 70.6 mm, vias 0 -> 4
- net /LED_FOG: track 0.00 -> 64.5 mm, vias 0 -> 2
- net /IN_WINDSHIELD_HEAT: track 7.31 -> 71.0 mm, vias 0 -> 2
- net /OLED_POWER_EN: track 0.00 -> 57.2 mm, vias 0 -> 4
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Other:
- board text added: "MIA EGV knowak.xyz & Jelcz Industries 03/2023"
