File: ecu/ecu.kicad_sch (KiCad schematic)
At the start: 85 parts, among them J1 INPUTS, J2 OUTPUTS, Q1 AOD4185, Q2 AOD4185, Q3 AOD4185, Q4 BXT3800P06M, Q5 BXT3800P06M, Q6 BXT3800P06M, Q7 BXT3800P06M, Q8 AOD4185, SW1 DISP_BUTTON, U1 MCP2551-I-SN, U2 L6981C33DR, U3 SN65HVD232, U4 ULN2003, U5 ULN2003

Commit message: stm dodany
Parts:
- added C29, C31, C32, C33, C34, C35: 1uF, symbol Device:C
- added C30: 100n, symbol Device:C
- added C36: 4.7u, symbol Device:C
- added U6: STM32F103VETx, Package_QFP:LQFP-100_14x14mm_P0.5mm, symbol MCU_ST_STM32F1:STM32F103VETx
Connections:
- net +3V3: now also C29.1, C31.1, C32.1, C33.1, C34.1, U6.100 (VDD), U6.11 (VDD), U6.22 (VDDA), U6.28 (VDD), U6.50 (VDD), U6.6 (VBAT), U6.75 (VDD)
- net GND: now also C30.2, U6.10 (VSS), U6.19 (VSSA), U6.27 (VSS), U6.49 (VSS), U6.74 (VSS), U6.94 (BOOT0), U6.99 (VSS)
- new net: C30.1, U6.14 (NRST)

Commit message: ecu schematic...
Parts:
- removed U3: SN65HVD232, Package_SO:SOIC-8_3.9x4.9mm_P1.27mm, symbol Interface_CAN_LIN:SN65HVD232
- added C2, C5: 18pF, symbol Device:C_Small
- added C42: 10uF 25V, symbol Device:C_Small
- added C6, C8: 1uF, symbol Device:C
- added C8: 100nF, symbol Device:C
- added D10, D11, D12, D13, D14, D15, D16, D17, D18, D19, D20, D21, D7, D8, D9: RED, symbol Device:LED
- added J2: DEBUG, symbol Connector_Generic:Conn_02x04_Odd_Even
- added J4: Conn_01x30_Socket, symbol Connector:Conn_01x30_Socket
- added R34, R35, R36, R37, R38, R39, R40, R41, R42, R43, R44, R45, R46, R47, R48: 220, symbol Device:R
- added R49, R51: 10k, symbol Device:R
- added R50: 100k, symbol Device:R
- added U2: L7805, symbol Regulator_Linear:L7805
- added Y1: 16MHz, Crystal:Crystal_SMD_3225-4Pin_3.2x2.5mm_HandSoldering, symbol Device:Crystal_GND24_Small
Connections:
- net +12V: now also C6.1, R50.1, U2.1 (IN)
- net +3V3: now also C35.1, C36.1, R49.1
- net +5V: now also C8.1, U2.3 (OUT)
- net CAN1_RX: now also U6.70 (PA11)
- net CAN1_TX: now also U6.71 (PA12)
- net GND: now also C29.2, C31.2, C32.2, C33.2, C34.2, C35.2, C36.2, C2.2, C42.1, C5.2, C6.2, C8.2, C8.2, D10.1 (K), D11.1 (K), D12.1 (K), D13.1 (K), D14.1 (K), D15.1 (K), D16.1 (K), D17.1 (K), D18.1 (K), D19.1 (K), D20.1 (K), D21.1 (K), D7.1 (K), D8.1 (K), D9.1 (K), J2.7 (Pin_7), J2.8 (Pin_8), J4.1 (Pin_1), J4.2 (Pin_2), J4.5 (Pin_5), R51.2, U2.2 (GND), Y1.2, Y1.4
- net at U6.12 (OSC_IN): now also C2.1, Y1.3
- net at U6.13 (OSC_OUT): now also C5.1, Y1.1
- net at C30.1, U6.14 (NRST): now also R49.2
- net VBAT_MEAS: now reaches U6.23 (PA0)
- net VBAT_MEAS: now also C8.1, R50.2, R51.1
- net USART1_TX: now reaches U6.68 (PA9)
- net USART1_TX: now also J2.5 (Pin_5)
- net USART1_RX: now reaches U6.69 (PA10)
- net USART1_RX: now also J2.3 (Pin_3)
- new net: D9.2 (A), R36.2
- new net: C42.2, J4.4 (Pin_4)
- new net: D8.2 (A), R35.2
- new net: D19.2 (A), R46.2
- new net: D11.2 (A), R38.2
- new net: D18.2 (A), R45.2
- new net: D17.2 (A), R44.2
- new net: D13.2 (A), R40.2
- new net: D14.2 (A), R41.2
- new net: D20.2 (A), R47.2
- new net: D16.2 (A), R43.2
- new net: D12.2 (A), R39.2
- new net: D10.2 (A), R37.2
- new net: D7.2 (A), R34.2
- new net: D21.2 (A), R48.2
- new net: D15.2 (A), R42.2
- new net +3.3V: J2.1 (Pin_1), J2.2 (Pin_2)
- new net LED_ABS: R41.1
- new net LED_AIRBAG: R40.1
- new net LED_BATTERY: R42.1, R48.1
- new net LED_BELT: R38.1
- new net LED_BRAKE: R37.1
- new net LED_CHARGING: R47.1
- new net LED_ELECTR: R35.1
- new net LED_FOG: R43.1
- new net LED_HEADLIGHT: R46.1
- new net LED_HEATER: R44.1
- new net LED_INDICATOR: R39.1
- new net LED_SIDELIGHTS: R45.1
- new net LED_STOP: R36.1
- new net LED_TEMP: R34.1
- new net SWDCLK: J2.6 (Pin_6)
- new net SWDIO: J2.4 (Pin_4)
Other:
- note added: "OLED"
- note added: "vcc"
- note added: "vcomh"
- note removed: "MCU low power mode"
- note removed: "RTC"
- note removed: "linia 5V"
- note removed: "na razie nie robię szyny 5V"
- moved on the sheet: C29, C31, C32, C33, C34, C35, C36

Commit message: pcb layout in progress
Parts:
- removed C12: 10uF 50V, symbol Device:C
- removed C13: 2.2uF, symbol Device:C_Small
- removed C15: 100nF, symbol Device:C_Small
- removed C18, C19: 22uF 10V, symbol Device:C
- removed C42: 10uF 25V, symbol Device:C_Small
- removed unit 4 of D3
- removed unit 5 of D3
- removed unit 3 of D3
- removed J4: Conn_01x30_Socket, symbol Connector:Conn_01x30_Socket
- removed L1: 33uH, symbol Device:L
- removed U2: L6981C33DR, Package_SO:SOIC-8-1EP_3.9x4.9mm_P1.27mm_EP2.514x3.2mm_ThermalVias, symbol krzysztof_lib:L6981
- removed U2: L7805, symbol Regulator_Linear:L7805
- added C12, C19, C47: 0.1uF, Capacitor_SMD:C_0603_1608Metric, symbol Device:C_Small
- added C16: 100n, Capacitor_SMD:C_0603_1608Metric, symbol Device:C_Small
- added C17, C48, C49, C50, C51: 10uF 25V, Capacitor_SMD:C_1206_3216Metric, symbol Device:C_Small
- added C42, C43: 10uF 25V, Capacitor_SMD:C_1206_3216Metric, symbol Device:C
- added C46: 100nF, Capacitor_SMD:C_0603_1608Metric, symbol Device:C
- added C54, C55: 22uF 10V, Capacitor_SMD:C_1206_3216Metric, symbol Device:C
- added D12: SK14WA, Diode_SMD:D_SOD-123F, symbol Device:D
- added D2 (x2): SK12WA, Diode_SMD:D_SOD-123F, symbol Device:D
- added D23: 1N4148, Diode_SMD:D_SOD-123, symbol Device:D
- added unit 3 of D6
- added unit 5 of D6
- added unit 4 of D6
- added F2: 250mA, Fuse:Fuse_0805_2012Metric, symbol Device:Polyfuse
- added J5: OLED, Connector_FFC-FPC:TE_3-1734839-0_1x30-1MP_P0.5mm_Horizontal, symbol Keithley197_OLED-rescue:Conn_01x30_Female-Connector
- added L2: 22uH 900mA, Inductor_SMD:L_Taiyo-Yuden_NR-50xx_HandSoldering, symbol Device:L
- added L3: 22uH, Inductor_SMD:L_Taiyo-Yuden_NR-50xx, symbol Device:L
- added R18, R19: 10k, Resistor_SMD:R_0603_1608Metric, symbol Device:R_Small
- added R20: 3k, Resistor_SMD:R_0603_1608Metric, symbol Device:R_Small
- added R54: 910k, Resistor_SMD:R_0603_1608Metric, symbol Device:R
- added R55: 50, Resistor_SMD:R_0603_1608Metric, symbol Device:R
- added R56, R57: 10k, Resistor_SMD:R_0603_1608Metric, symbol Device:R
- added R8: 29k, Resistor_SMD:R_0603_1608Metric, symbol Device:R
- added R9: 1k, Resistor_SMD:R_0603_1608Metric, symbol Device:R
- added U1: SB6286, Package_TO_SOT_SMD:SOT-23-6, symbol Regulator_Switching:MT3608
- added U3: AOZ1282CI-1, Package_TO_SOT_SMD:SOT-23-6, symbol Regulator_Switching:AOZ1282CI-1
- added U4: 78L15MG-AA3-R, Package_TO_SOT_SMD:SOT-223-3_TabPin2, symbol Regulator_Linear:L7815
- added U7: AMS1117-5.0, Package_TO_SOT_SMD:SOT-223-3_TabPin2, symbol Regulator_Linear:AMS1117-5.0
- added U9: FM24CL16B, Package_SO:SOIC-8_3.9x4.9mm_P1.27mm, symbol Memory_NVRAM:FM24C64B
- C1: value 100uF 50V -> 100uF 25V; footprint (none) -> Capacitor_SMD:CP_Elec_8x6.2
- C10, C11, C14, C16, C17, C2, C20, C21, C22, C23, C24, C25, C26, C27, C28, C29, C3, C30, C31, C33, C34, C35, C36, C4, C5, C6, C7, C8, C9: footprint (none) -> Capacitor_SMD:C_0603_1608Metric
- C32: value 1uF -> 10uF 25V; footprint (none) -> Capacitor_SMD:C_1206_3216Metric
- D10, D11, D12, D13, D14, D15, D16, D17, D18, D19, D20, D21, D7, D8, D9: footprint (none) -> LED_SMD:LED_0805_2012Metric_Pad1.15x1.40mm_HandSolder
- F1: footprint (none) -> Fuse:Fuse_0805_2012Metric
- J1: footprint (none) -> Connector_Molex:Molex_Mini-Fit_Jr_5566-24A_2x12_P4.20mm_Vertical
- J2: footprint (none) -> Connector_IDC:IDC-Header_2x04_P2.54mm_Vertical
- J2: footprint (none) -> Connector_Molex:Molex_Mini-Fit_Jr_5566-22A_2x11_P4.20mm_Vertical
- R1, R10, R11, R12, R13, R14, R15, R16, R17, R18, R19, R2, R20, R21, R22, R23, R24, R25, R26, R27, R28, R29, R3, R30, R31, R32, R33, R34, R35, R36, R37, R38, R39, R4, R40, R41, R42, R43, R44, R45, R46, R47, R48, R49, R5, R50, R51, R6, R7, R8, R9: footprint (none) -> Resistor_SMD:R_0603_1608Metric
- SW1: footprint (none) -> Button_Switch_THT:SW_PUSH_6mm_H13mm
- U4, U5: footprint (none) -> Package_SO:SOP-16_3.9x9.9mm_P1.27mm
Connections:
- net +12V: now also F2.2; no longer C1.1, C6.1
- net +3.3V: now also C46.1, R56.1, R57.1, U9.8 (VDD)
- net +3V3: now also C51.1, J5.24 (Pin_24), J5.26 (Pin_26); no longer C32.1
- net +5V: now also U7.2 (VO)
- net APC: now also U4.7 (I7); no longer U5.5 (I5)
- net BMS: now also U4.1 (I1); no longer U4.4 (I4)
- net BMS_L: now also U4.16 (O1); no longer U4.13 (O4)
- net GND: now also C12.2, C17.2, C19.2, C42.2, C43.2, C46.2, C47.2, C48.2, C49.2, C50.2, C51.2, C54.2, C55.2, D12.2 (A), D2.2 (A), D23.1 (K), J5.1 (Pin_1), J5.10 (Pin_10), J5.14 (Pin_14), J5.15 (Pin_15), J5.16 (Pin_16), J5.17 (Pin_17), J5.2 (Pin_2), J5.28 (Pin_28), J5.30 (Pin_30), J5.5 (Pin_5), J5.6 (Pin_6), J5.7 (Pin_7), J5.8 (Pin_8), J5.9 (Pin_9), R20.1, R54.1, R9.1, U1.2 (GND), U3.2 (GND), U4.2 (GND), U7.1 (GND), U9.1 (A0), U9.2 (A1), U9.3 (A2), U9.4 (VSS), U9.7 (WP)
- net HEATING: now also U5.5 (I5); no longer U5.4 (I4)
- net INDIC_LEFT: now also U5.1 (I1); no longer U4.6 (I6)
- net INDIC_RIGHT: now also U5.2 (I2); no longer U4.5 (I5)
- net INVERTER: now also U4.4 (I4); no longer U4.3 (I3)
- net INVERTER_L: now also U4.13 (O4); no longer U4.14 (O3)
- net IN_AIRBAG: now also D6.6 (K5); no longer D6.1 (K1)
- net IN_CRASH: now also D5.1 (K1); no longer D5.5 (K4)
- net IN_DF_CONV: now also D6.4 (K3)
- net IN_DRIVE_DIR_2: now also D6.3 (K2)
- net IN_HIGHBEAM: now also D5.5 (K4); no longer D5.1 (K1)
- net IN_KEY1: now also D5.4 (K3); no longer D6.3 (K2)
- net IN_KEY2: now also D5.3 (K2); no longer D5.4 (K3)
- net IN_PARK: now also D6.5 (K4); no longer D5.3 (K2)
- net IN_WINDSHIELD_JET: now also D6.1 (K1)
- net LED_BATTERY: no longer R48.1
- net LIGHT_DAYTIME: now also U4.6 (I6); no longer U5.2 (I2)
- net LIGHT_HAZARD: now also U4.5 (I5); no longer U5.3 (I3)
- net LIGHT_REVERSE: now also U5.4 (I4); no longer U5.1 (I1)
- net LIGHT_STOP: now also U5.3 (I3); no longer U4.7 (I7)
- net SWDCLK: now also U6.76 (PA14)
- net SWDIO: now also U6.72 (PA13)
- net THR1: now also U6.24 (PA1)
- net THR2: now also U6.25 (PA2)
- net WINDSHIELD_HEAT: now also U4.3 (I3); no longer U4.1 (I1)
- net WINDSHIELD_HEAT_L: now also U4.14 (O3); no longer U4.16 (O1)
- net at R30.2, U5.14 (O3): now also Q8.1 (G); no longer Q5.1 (G)
- net at R32.2, U5.12 (O5): now also Q6.1 (G); no longer Q7.1 (G)
- net at R31.2, U5.13 (O4): now also Q3.1 (G); no longer Q6.1 (G)
- net at R29.2, U5.15 (O2): now also Q1.1 (G); no longer Q4.1 (G)
- net at R28.2, U5.16 (O1): now also Q2.1 (G); no longer Q3.1 (G)
- net at R27.2, U4.11 (O6): now also Q4.1 (G); no longer Q2.1 (G)
- net at F1.1: now also C54.1, C55.1, L2.2, R19.2
- net at R33.2, U4.10 (O7): now also Q7.1 (G); no longer Q8.1 (G)
- net OLED_CS: now reaches U6.26 (PA3)
- net OLED_CS: now also J5.19 (Pin_19)
- net OLED_DC: now reaches U6.29 (PA4)
- net OLED_DC: now also J5.18 (Pin_18)
- net OLED_SCK: now reaches U6.30 (PA5)
- net OLED_SCK: now also J5.13 (Pin_13)
- net OLED_RES: now reaches U6.31 (PA6)
- net OLED_RES: now also J5.20 (Pin_20)
- net OLED_MOSI: now reaches U6.32 (PA7)
- net OLED_MOSI: now also J5.12 (Pin_12)
- net SCL: now reaches U6.92 (PB6)
- net SCL: now also R57.2, U9.6 (SCL)
- net SDA: now reaches U6.93 (PB7)
- net SDA: now also R56.2, U9.5 (SDA)
- net at R26.2, U4.12 (O5): now also Q5.1 (G); no longer Q1.1 (G)
- new net: C16.2, U3.1 (BST)
- new net: R19.1, R20.2, U3.3 (FB)
- new net: R18.1, U3.4 (EN)
- new net: C1.1, C32.1, C42.1, C43.1, C6.1, D2.1 (K), F2.1, L3.1, R18.2, U1.5 (IN), U3.5 (VIN), U7.3 (VI)
- new net: C16.1, D12.1 (K), L2.1, U3.6 (LX)
- new net: C17.1, C19.1, D2.1 (K), R8.2, U4.1 (IN)
- new net: D23.2 (A), R55.1
- new net: J5.27 (Pin_27), R55.2
- new net: R8.1, R9.2, U1.3 (FB)
- new net: C49.1, J5.25 (Pin_25)
- new net: D2.2 (A), L3.2, U1.1 (SW)
- new net: C48.1, J5.4 (Pin_4)
- new net: J5.22 (Pin_22), R54.2
- new net +15V: C12.1, C47.1, C50.1, J5.29 (Pin_29), J5.3 (Pin_3), U4.3 (OUT)
- new net LED_BATTERY_HV: R48.1
- new net OLED_POWER_EN: U1.4 (EN)
- no-connect marks 12 -> 15
Other:
- note removed: "OLED"
- note removed: "TVS i filtr common mode?"
- note removed: "vcc"
- note removed: "vcomh"
- note removed: "wolne SPI pod OLEDa"
- moved on the sheet: C1, C14, C6, C8, D4, D5A, D5B, D5C, D5D, D6A, D6B, F1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

Commit message: pcb layout completed
Connections:
- net +3.3V is gone; now on net +3V3: C46.1, J2.1 (Pin_1), J2.2 (Pin_2), R56.1, R57.1, U9.8 (VDD)
- net +3V3: now also U6.21 (VREF+)
- net APC: now also U6.17 (PC2)
- net BMS: now also U6.35 (PB0)
- net GND: now also U6.20 (VREF-)
- net HEATING: now also U6.40 (PE9)
- net INDIC_LEFT: now also U6.36 (PB1)
- net INDIC_RIGHT: now also U6.37 (PB2)
- net INVERTER: now also U6.18 (PC3)
- net IN_AIRBAG: now also U6.87 (PD6)
- net IN_BRAKE_1: now also U6.55 (PD8)
- net IN_CEINT: now also U6.45 (PE14)
- net IN_CRASH: now also U6.89 (PB3)
- net IN_CTL_APC: now also U6.46 (PE15)
- net IN_DF_CONV: now also U6.85 (PD4)
- net IN_DISP: now also U6.44 (PE13)
- net IN_DRIVE_DIR_1: now also U6.51 (PB12)
- net IN_DRIVE_DIR_2: now also U6.84 (PD3)
- net IN_ECO: now also U6.47 (PB10)
- net IN_FOG_LIGHT: now also U6.53 (PB14)
- net IN_HIGHBEAM: now also U6.91 (PB5)
- net IN_INDICATOR_RIGHT: now also U6.56 (PD9)
- net IN_KEY1: now also U6.90 (PB4)
- net IN_KEY2: now also U6.88 (PD7)
- net IN_PARK: now also U6.86 (PD5)
- net IN_SIDELIGHTS: now also U6.54 (PB15)
- net IN_WINDSHIELD_HEAT: now also U6.48 (PB11)
- net IN_WINDSHIELD_JET: now also U6.83 (PD2)
- net IN_WIPER: now also U6.52 (PB13)
- net LED_ABS: now also U6.3 (PE4)
- net LED_AIRBAG: now also U6.2 (PE3)
- net LED_BATTERY: now also U6.98 (PE1)
- net LED_BATTERY_HV: now also U6.42 (PE11)
- net LED_BELT: now also U6.4 (PE5)
- net LED_BRAKE: now also U6.5 (PE6)
- net LED_CHARGING: now also U6.41 (PE10)
- net LED_ELECTR: now also U6.8 (PC14)
- net LED_FOG: now also U6.97 (PE0)
- net LED_HEADLIGHT: now also U6.58 (PD11)
- net LED_HEATER: now also U6.96 (PB9)
- net LED_INDICATOR: now also U6.1 (PE2)
- net LED_SIDELIGHTS: now also U6.57 (PD10)
- net LED_STOP: now also U6.7 (PC13)
- net LED_TEMP: now also U6.9 (PC15)
- net LIGHT_DAYTIME: now also U6.16 (PC1)
- net LIGHT_HAZARD: now also U6.15 (PC0)
- net LIGHT_REVERSE: now also U6.39 (PE8)
- net LIGHT_STOP: now also U6.38 (PE7)
- net OLED_POWER_EN: now also U6.43 (PE12)
- net WINDSHIELD_HEAT: now also U6.33 (PC4)
- net WIPERS: now also U6.34 (PC5)
- no-connect marks 15 -> 30
Other:
- moved on the sheet: C2, C5, Y1

Commit message: pcb layout completed
Other:
- note removed: "polakierować PCB"
Changed lines of the file:
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@@
     (effects (font (size 1.27 1.27)) (justify left bottom))
-  )
-  (text "polakierować PCB" (at 323.85 254 0)
-    (effects (font (size 5 5)) (justify left bottom))
   )
   (label "IN_KEY2" (at 213.995 316.23 0) (fields_autoplaced)

Commit message: remove build
Parts:
- C17, C32, C42, C43, C48, C49, C50, C51: TME (none) -> CL31A106MAHNNNE
- D1, D2, D3, D5, D6: TME (none) -> PESD3V3L5UY.115
- D4: TME (none) -> BZT52C3V6-13-F
- F1, F2: value 250mA -> 350mA; TME (none) -> SR035-06
- J1: TME (none) -> MX-5566-24A
- J5: TME (none) -> F0500WR-S-30PT
- L2: LCSC (none) -> C222921; MPN (none) -> NRS5020T220MMGJ; code NRS5020T220MMGJ -> (none)
- Q1, Q2, Q3, Q8: TME (none) -> AOD4185
- Q4, Q5, Q6, Q7: TME (none) -> BXT3800P06M
- U1: TME (none) -> MCP2551-E/SN
- U4: TME (none) -> DI78L15UAB-DIO
- U4, U5: TME (none) -> ULN2003ADR
- Y1: TME (none) -> 3225-16M-SR
